File: macropad/macropad.kicad_pcb (KiCad board)
At the start: 2 copper layers, 88.1 x 61.9 mm, 19 parts, among them U1 Arduino_Pro_Micro

Commit message: change pro micro to seeed studio xiao
Parts:
- U1: value Arduino_Pro_Micro -> XIAO-RP2040-DIP; footprint ScottoKeebs_MCU:Arduino_Pro_Micro -> OPL:XIAO-RP2040-DIP
- moved U1 10.9 mm to (166.5, 65.4)
Connections:
- U1 pad 1: unconnected-(U1-TX0/PD3-Pad1) -> Column 0
- U1 pad 10: Row 2 -> unconnected-(U1-GPIO4/MISO-Pad10)
- U1 pad 2: unconnected-(U1-RX1/PD2-Pad2) -> Column 1
- U1 pad 3: unconnected-(U1-GND-Pad3) -> Column 2
- U1 pad 4: unconnected-(U1-GND-Pad4) -> Row 0
- U1 pad 5: Column 0 -> Row 1
- U1 pad 6: Column 1 -> Row 2
- U1 pad 7: Column 2 -> unconnected-(U1-GPIO0/TX-Pad7)
- U1 pad 8: Row 0 -> unconnected-(U1-GPIO1/RX-Pad8)
- U1 pad 9: Row 1 -> unconnected-(U1-GPIO2/SCK-Pad9)
Routing:
- net Row 2: track 64.5 -> 78.2 mm
- net Row 1: track 50.1 -> 61.7 mm
- net Column 2: track 65.9 -> 74.4 mm
- net Row 0: track 52.6 -> 45.3 mm
- net Column 1: track 88.3 -> 91.2 mm
- net Column 0: track 111.3 -> 114.2 mm
- removed copper zone on B.Cu, net (none)
- removed copper zone on F.Cu, net (none)
Other:
- board size 88.1 x 61.9 mm -> 85.7 x 61.9 mm
- board text added: "By Ayaan Grover"
- board text added: "NINEFOLD"
